Commit message: update assets

File: assets/robots/allegro_hand/allegro_hand_right_retargeting_base.urdf (robot description, URDF)
Before this commit: robot allegro_right, 29 links, 28 joints
Joints:
- joint joint_0.0: origin xyz=0.0 0.0435 -0.001542 rpy=-0.08726646255000003 -0.0 0.0 -> xyz=0.0 0.0435 -0.001542 rpy=-0.08726646254999999 -0.0 0.0
- joint joint_12.0: origin xyz=-0.0182 0.019333 -0.045987 rpy=3.141592653589793 -1.483529865139793 1.5707963276897932 -> xyz=-0.0182 0.019333 -0.045987 rpy=3.141592653589793 -1.4835298651397932 1.5707963276897934
- joint joint_8.0: origin xyz=0.0 -0.0435 -0.001542 rpy=0.08726646255000003 -0.0 0.0 -> xyz=0.0 -0.0435 -0.001542 rpy=0.08726646254999999 -0.0 0.0
